File: STM32F1_FOC_TransistorDriven/STM32F1_FOC.kicad_sch (KiCad schematic)
At the start: 93 parts, among them IC1 MP9486A, J1 Screw_Terminal_01x01, J11 Screw_Terminal_01x01, J12 Screw_Terminal_01x01, J13 Conn_01x03, J14 Screw_Terminal_01x01, J15 Screw_Terminal_01x01, J17 Conn_01x03, J18 Conn_01x03, J19 Conn_01x04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

Commit message: Design 4 layer Board with separate supply and ground plane
Note:
Below points WIP...
-Need to check all the plane.
-Place ground via if needed near to shunt and return path of the supply.
-Validate the layout.
Parts:
- R12: footprint Footprints:R_0603 -> Jumper:SolderJumper-2_P1.3mm_Open_Pad1.0x1.5mm
Changed lines of the file:
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@@
 			)
 		)
-		(property "Footprint" "Footprints:R_0603"
+		(property "Footprint" "Jumper:SolderJumper-2_P1.3mm_Open_Pad1.0x1.5mm"
 			(at 176.53 62.738 90)
 			(effects
